File: Esp32 Can+IMU/Esp32 Can+IMU.kicad_sch (KiCad schematic)
At the start: 88 parts, among them J1 Conn_01x04_Pin, J11 Qwiic_Vertical, J12 USB_C_Receptacle_USB2.0_16P, J2 Conn_01x04_Pin, J4 PINHD_1x3_Male, J5 PINHD_1x3_Male, J6 PINHD_1x3_Male, J7 PINHD_1x3_Male, J8 PINHD_1x3_Male, J9 PINHD_1x3_Male, SW1 SMD_4.2x3.2mm_h2.5mm, SW2 SMD_4.2x3.2mm_h2.5mm, U1 ESP32-S3-WROOM-1, U2 ISM6HG256XTR, U3 SN65HVD230DR, U4 TPS54360BQDDARQ1, U5 AP2112K-3.3, U6 USBLC6-2P6

Commit message: Update ESP32 CAN IMU board revision
Parts:
- removed 3v3/2: CAN_VREF, TestPoint:TestPoint_THTPad_1.0x1.0mm_Drill0.5mm, symbol Connector:TestPoint
- removed D2: SS54, Diode_SMD:D_SMA, symbol Device:D_Schottky
- removed J12: USB_C_Receptacle_USB2.0_16P, Connector_USB:USB_C_Receptacle_G-Switch_GT-USB-7051x, symbol Connector:USB_C_Receptacle_USB2.0_16P
- removed J4, J5, J6: PINHD_1x3_Male, Connector_PinHeader_2.54mm:PinHeader_1x03_P2.54mm_Vertical, symbol PCM_SL_Pin_Headers:PINHD_1x3_Male
- removed JP2, JP3, JP4: 3v3 input, Jumper:SolderJumper-2_P1.3mm_Open_RoundedPad1.0x1.5mm, symbol Jumper:SolderJumper_2_Open
- removed R16, R17: 10kΩ, Resistor_SMD:R_0402_1005Metric, symbol Device:R_US
- removed R7, R8: 5.1kΩ, Resistor_SMD:R_0402_1005Metric, symbol Device:R_US
- removed TP_5v1: 5v, TestPoint:TestPoint_THTPad_1.0x1.0mm_Drill0.5mm, symbol Connector:TestPoint
- removed TP_GND1: GND, TestPoint:TestPoint_THTPad_1.0x1.0mm_Drill0.5mm, symbol Connector:TestPoint
- removed U6: USBLC6-2P6, Package_TO_SOT_SMD:SOT-666, symbol Power_Protection:USBLC6-2P6
- added J10: PWM4, Connector:PinHeader_1x03_P2.54mm_Vertical_Close, symbol PCM_SL_Pin_Headers:PINHD_1x3_Male
- added J12: ADC1, Connector:PinHeader_1x03_P2.54mm_Vertical_Close, symbol PCM_SL_Pin_Headers:PINHD_1x3_Male
- added J13: ADC2, Connector:PinHeader_1x03_P2.54mm_Vertical_Close, symbol PCM_SL_Pin_Headers:PINHD_1x3_Male
- added J14: ADC3, Connector:PinHeader_1x03_P2.54mm_Vertical_Close, symbol PCM_SL_Pin_Headers:PINHD_1x3_Male
- added J15: ADC4, Connector:PinHeader_1x03_P2.54mm_Vertical_Close, symbol PCM_SL_Pin_Headers:PINHD_1x3_Male
- added J3: UART0, Connector_JST:JST_GH_SM03B-GHS-TB_1x03-1MP_P1.25mm_Horizontal, symbol Connector_Generic:Conn_01x03
- added J4: UART1, Connector_JST:JST_GH_SM03B-GHS-TB_1x03-1MP_P1.25mm_Horizontal, symbol Connector_Generic:Conn_01x03
- added J5: USB, Connector_JST:JST_GH_SM03B-GHS-TB_1x03-1MP_P1.25mm_Horizontal, symbol Connector_Generic:Conn_01x03
- added J6: 5V ⏚, Connector_PinHeader_2.54mm:PinHeader_1x02_P2.54mm_Vertical, symbol Connector_Generic:Conn_01x02
- added TP_SDO1: SDO, TestPoint:TestPoint_Pad_D1.0mm, symbol Connector:TestPoint
- Boot2: renamed from SW2; value SMD_4.2x3.2mm_h2.5mm -> BOOT
- CAND1, CANR1: footprint TestPoint:TestPoint_THTPad_1.0x1.0mm_Drill0.5mm -> TestPoint:TestPoint_Pad_1.0x1.0mm
- CAN_TERM1: value CAN_TERM -> CAN 120R
- D3: value Green -> PWR
- D4: value Red -> LIFE
- H1, H2, H3, H4: value MountingHole -> M3; footprint MountingHole:MountingHole_3.2mm_M3_ISO7380_Pad -> MountingHole:MountingHole_3.2mm_M3_Pad_Via
- J1: value Conn_01x04_Pin -> CAN0
- J11: value Qwiic_Vertical -> Qwiic
- J2: value Conn_01x04_Pin -> CAN1
- J7: value PINHD_1x3_Male -> PWM1; footprint Connector_PinHeader_2.54mm:PinHeader_1x03_P2.54mm_Vertical -> Connector:PinHeader_1x03_P2.54mm_Vertical_Close
- J8: value PINHD_1x3_Male -> PWM2; footprint Connector_PinHeader_2.54mm:PinHeader_1x03_P2.54mm_Vertical -> Connector:PinHeader_1x03_P2.54mm_Vertical_Close
- J9: value PINHD_1x3_Male -> PWM3; footprint Connector_PinHeader_2.54mm:PinHeader_1x03_P2.54mm_Vertical -> Connector:PinHeader_1x03_P2.54mm_Vertical_Close
- R1: value 523k -> 174k
- R12, R13, R14: value 33Ω -> 33
- R15: value 10kΩ -> 33
- R18, R19: value 4.7kΩ -> 4.7k
- R2: value 84.5kΩ -> 35.3k
- R3: value 162kΩ -> 162k
- R4: value 13.0kΩ -> 13.0k
- R5: value 59kΩ -> 59k
- R6: value 10.2kΩ -> 10.2k
- R7: renamed from Reset1; value 10kΩ -> 10k
- R8: renamed from Boot1; value 10kΩ -> 10k
- R9: value 120Ω -> 120
- Reset1: renamed from SW1; value SMD_4.2x3.2mm_h2.5mm -> RESET
- TP_3v3: footprint TestPoint:TestPoint_THTPad_1.0x1.0mm_Drill0.5mm -> TestPoint:TestPoint_THTPad_D1.0mm_Drill0.5mm
- TP_CS1: value IMU CS -> CS1; footprint TestPoint:TestPoint_THTPad_1.0x1.0mm_Drill0.5mm -> TestPoint:TestPoint_Pad_D1.0mm
- TP_INT1: value IMU INT1 -> INT1; footprint TestPoint:TestPoint_THTPad_1.0x1.0mm_Drill0.5mm -> TestPoint:TestPoint_Pad_D1.0mm
- TP_INT2: value IMU INT2 -> INT2; footprint TestPoint:TestPoint_THTPad_1.0x1.0mm_Drill0.5mm -> TestPoint:TestPoint_Pad_D1.0mm
- TP_SCL1: value IMU SCL -> SCL1; footprint TestPoint:TestPoint_THTPad_1.0x1.0mm_Drill0.5mm -> TestPoint:TestPoint_Pad_D1.0mm
- TP_SDA1: value IMU_SDA -> SDA1; footprint TestPoint:TestPoint_THTPad_1.0x1.0mm_Drill0.5mm -> TestPoint:TestPoint_Pad_D1.0mm
- XT30F1, XT30F2: value Conn_01x02 -> XT30F
- XT30M1: value Conn_01x02 -> XT30M
Connections:
- net ADC_3 is gone; now on an unnamed net: U1.15 (IO3)
- net +3.3V: now also J12.2, J13.2, J14.2, J15.2
- net +5V: now also J10.2, J6.2 (Pin_2)
- net GND: now also D_TVS1.2 (A), J10.3, J12.3, J13.3, J14.3, J15.3, J3.2 (Pin_2), J4.2 (Pin_2), J5.1 (Pin_1), J6.1 (Pin_1); no longer D_TVS1.1 (K)
- net PWM_1: now also U1.22 (IO14); no longer U1.4 (IO4)
- net PWM_2: now also U1.21 (IO13); no longer U1.5 (IO5)
- net PWM_3: now also U1.20 (IO12); no longer U1.6 (IO6)
- net SDO/TA0: now also TP_SDO1.1
- net USB_D+: now also J5.2 (Pin_2)
- net USB_D-: now also J5.3 (Pin_3)
- net at F1.1, XT30F1.2 (Pin_2), XT30F2.2 (Pin_2)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: now also D_TVS1.1 (K); no longer D_TVS1.2 (A)
- net at R15.2: now also J10.1
- net at R23.2: no longer U1.8 (IO15)
- net PWM_4: now reaches U1.19 (IO11)
- net PWM_4: now also R15.1
- net UART1RX: now reaches U1.34 (IO41)
- net UART1RX: now also J4.3 (Pin_3)
- net UART1TX: now reaches U1.35 (IO42)
- net UART1TX: now also J4.1 (Pin_1)
- net UART0RX: now reaches U1.36 (RXD0)
- net UART0RX: now also J3.3 (Pin_3)
- net UART0TX: now reaches U1.37 (TXD0)
- net UART0TX: now also J3.1 (Pin_1)
- net ADC1_CH6: now reaches U1.7 (IO7)
- net ADC1_CH6: now also J15.1
- net AD2_1: no longer names the net of U1.38 (IO2)
- net ADC_1: no longer names the net of U1.39 (IO1)
- net ADC_1: no longer R15.1
- net CANH renamed CAN+
- net CANL renamed CAN-
- new net ADC1_CH0: J13.1, U1.5 (IO5)
- new net ADC1_CH1: J12.1, U1.4 (IO4)
- new net ADC1_CH5: J14.1, U1.6 (IO6)
- no-connect marks 18 -> 10
Other:
- moved on the sheet: Boot2, C15, C3, D4, D_TVS1, J7, J8, J9, R12, R13, R14, R23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

Commit message: updated schematic with pogo pads
Parts:
- removed Boot2: BOOT, PCM_SparkFun-Switch:Push_SMD_4.2x3.2mm, symbol PCM_SparkFun-Switch:SPST_Push_SMD_4.2x3.2mm_h2.5mm
- removed CAND1: CAN_D, TestPoint:TestPoint_Pad_1.0x1.0mm, symbol Connector:TestPoint
- removed CANR1: CAN_R, TestPoint:TestPoint_Pad_1.0x1.0mm, symbol Connector:TestPoint
- removed D6: SS54, Diode_SMD:D_SMA, symbol Device:D_Schottky
- removed J3: UART0, Connector_JST:JST_GH_SM03B-GHS-TB_1x03-1MP_P1.25mm_Horizontal, symbol Connector_Generic:Conn_01x03
- removed J5: USB, Connector_JST:JST_GH_SM03B-GHS-TB_1x03-1MP_P1.25mm_Horizontal, symbol Connector_Generic:Conn_01x03
- removed Reset1: RESET, PCM_SparkFun-Switch:Push_SMD_4.2x3.2mm, symbol PCM_SparkFun-Switch:SPST_Push_SMD_4.2x3.2mm_h2.5mm
- removed TP_CS1: CS1, TestPoint:TestPoint_Pad_D1.0mm, symbol Connector:TestPoint
- removed TP_INT1: INT1, TestPoint:TestPoint_Pad_D1.0mm, symbol Connector:TestPoint
- removed TP_INT2: INT2, TestPoint:TestPoint_Pad_D1.0mm, symbol Connector:TestPoint
- removed TP_SCL1: SCL1, TestPoint:TestPoint_Pad_D1.0mm, symbol Connector:TestPoint
- removed TP_SDA1: SDA1, TestPoint:TestPoint_Pad_D1.0mm, symbol Connector:TestPoint
- removed TP_SDO1: SDO, TestPoint:TestPoint_Pad_D1.0mm, symbol Connector:TestPoint
- added CAN_5V_PWR1: 5V_PWR, Jumper:SolderJumper-2_P1.3mm_Open_RoundedPad1.0x1.5mm, symbol Jumper:SolderJumper_2_Open
- added CAN_Vin_PWR1: Vin_PWR, Jumper:SolderJumper-2_P1.3mm_Open_RoundedPad1.0x1.5mm, symbol Jumper:SolderJumper_2_Open
- added D10, D9: SS54, Diode_SMD:D_SMA, symbol Device:D_Schottky
- added D6: FAULT, LED_SMD:LED_0603_1608Metric, symbol PCM_SparkFun-LED:LED_Blue_0603
- added J17: USB_C_Receptacle_USB2.0_16P, Connector_USB:USB_C_Receptacle_JAE_DX07S016JA1R1500, symbol Connector:USB_C_Receptacle_USB2.0_16P
- added J3, J5: Conn_01x09_Pin, Pogo:Untitled, symbol Connector:Conn_01x09_Pin
- added R10, R11: 5.1k, Resistor_SMD:R_0402_1005Metric, symbol Device:R_US
- added R24: 100Ω, Resistor_SMD:R_0402_1005Metric, symbol Device:R_US
- added U6: USBLC6-2SC6, Package_TO_SOT_SMD:SOT-666, symbol Power_Protection:USBLC6-2SC6
- J4: now fitted
Connections:
- net +3.3V: now also J3.2 (Pin_2), J5.2 (Pin_2)
- net +5V: now also CAN_5V_PWR1.1 (A), CAN_Vin_PWR1.1 (A), D9.1 (K), U6.5 (VBUS)
- net CAN_D: now also J3.4 (Pin_4)
- net CAN_R: now also J3.3 (Pin_3)
- net CS: now also J5.6 (Pin_6)
- net GND: now also D6.1 (K), J17.A1 (GND), J17.A12 (GND), J17.B1 (GND), J17.B12 (GND), J17.SH (SHIELD), J3.1 (Pin_1), J3.5 (Pin_5), J5.1 (Pin_1), J5.5 (Pin_5), R10.2, R11.2, U6.2 (GND)
- net INT1: now also J5.8 (Pin_8)
- net INT2: now also J5.9 (Pin_9)
- net SCL: now also J5.3 (Pin_3)
- net SDA: now also J5.4 (Pin_4)
- net SDO/TA0: now also J5.7 (Pin_7)
- net UART0RX: now also J3.8 (Pin_8)
- net UART0TX: now also J3.9 (Pin_9)
- net USB_D+: now also U6.4 (I/O2)
- net USB_D-: now also U6.6 (I/O1)
- net at J1.1 (Pin_1), J2.1 (Pin_1): now also D10.1 (K)
- net STATUS: now reaches R23.2, U1.15 (IO3)
- net RESET: now reaches C3.2, R7.2, U1.3 (EN)
- net RESET: now also J3.6 (Pin_6)
- net BOOT: now reaches C15.2, R8.1, U1.27 (IO0)
- net BOOT: now also J3.7 (Pin_7)
- net FAULT: now reaches U1.38 (IO2)
- net FAULT: now also R24.2
- new net: CAN_5V_PWR1.2 (B), CAN_Vin_PWR1.2 (B), D10.2 (A)
- new net: J17.A8 (SBU1), R10.1
- new net: J17.B8 (SBU2), R11.1
- new net: D9.2 (A), J17.A4 (VBUS), J17.A9 (VBUS), J17.B4 (VBUS), J17.B9 (VBUS)
- new net: J17.A6 (D+), J17.B6 (D+), U6.3 (I/O2)
- new net: J17.A7 (D-), J17.B7 (D-), U6.1 (I/O1)
- new net: D6.2 (A), R24.1
Other:
- moved on the sheet: C11, C14, D3, D4, D7, D_TVS1, F1, H1, H2, H3, H4, J6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

Commit message: hand soldering usbLC6
Parts:
- removed U6: USBLC6-2SC6, Package_TO_SOT_SMD:SOT-666, symbol Power_Protection:USBLC6-2SC6
- added U7: USBLC6-2SC6, Package_TO_SOT_SMD:SOT-23-6_Handsoldering, symbol Power_Protection:USBLC6-2SC6
Connections:
- net +5V: now also U7.5 (VBUS)
- net GND: now also U7.2 (GND)
- net USB_D+: now also U7.4 (I/O2)
- net USB_D-: now also U7.6 (I/O1)
- net at J17.A6 (D+), J17.B6 (D+): now also U7.3 (I/O2)
- net at J17.A7 (D-), J17.B7 (D-): now also U7.1 (I/O1)
Changed lines of the file:
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@@
 	(wire
 		(pts
+			(xy 255.27 292.1) (xy 255.27 293.37)
+		)
+		(stroke
+			(width 0)
+			(type default)
+		)
+	)
+	(wire
+		(pts
 			(xy 63.5 261.62) (xy 63.5 270.51)
 		)
@@
 	(wire
 		(pts
+			(xy 255.27 294.64) (xy 255.27 298.45)
+		)
+		(stroke
+			(width 0)
+			(type default)
+		)
+	)
+	(wire
+		(pts
 			(xy 78.74 314.96) (xy 72.39 314.96)
 		)
@@
 	(wire
 		(pts
-			(xy 255.27 293.37) (xy 255.27 292.1)
-		)
-		(stroke
-			(width 0)
-			(type default)
-		)
-	)
-	(wire
-		(pts
 			(xy 181.61 248.92) (xy 184.15 248.92)
 		)
@@
 	(wire
 		(pts
-			(xy 255.27 298.45) (xy 255.27 294.64)
-		)
-		(stroke
-			(width 0)
-			(type default)
-		)
-	)
-	(wire
-		(pts
 			(xy 118.11 256.54) (xy 132.08 256.54)
 		)
@@
 	)
 	(symbol
+		(lib_id "Power_Protection:USBLC6-2SC6")
+		(at 260.35 292.1 0)
+		(unit 1)
+		(body_style 1)
+		(exclude_from_sim no)
+		(in_bom yes)
+		(on_board yes)
+		(in_pos_files yes)
+		(dnp no)
+		(fields_autoplaced yes)
+		(property "Reference" "U7"
+			(at 262.0011 284.48 0)
+			(show_name no)
+			(do_not_autoplace no)
+			(effects
+				(font
+					(size 1.27 1.27)
+				)
+				(justify left)
+			)
+		)
+		(property "Value" "USBLC6-2SC6"
+			(at 262.0011 287.02 0)
+			(show_name no)
+			(do_not_autoplace no)
+			(effects
+				(font
+					(size 1.27 1.27)
+				)
+				(justify left)
+			)
+		)
+		(property "Footprint" "Package_TO_SOT_SMD:SOT-23-6_Handsoldering"
+			(at 261.62 298.45 0)
+			(hide yes)
+			(show_name no)
+			(do_not_autoplace no)
+			(effects
+				(font
+					(size 1.27 1.27)
+					(italic yes)
+				)
+				(justify left)
+			)
+		)
+		(property "Datasheet" "https://www.st.com/resource/en/datasheet/usblc6-2.pdf"
+			(at 261.62 300.355 0)
+			(hide yes)
+			(show_name no)
+			(do_not_autoplace no)
+			(effects
+				(font
+					(size 1.27 1.27)
+				)
+				(justify left)
+			)
+		)
+		(property "Description" "Very low capacitance ESD protection diode, 2 data-line, SOT-23-6"
+			(at 260.35 292.1 0)
+			(hide yes)
+			(show_name no)
+			(do_not_autoplace no)
+			(effects
+				(font
+					(size 1.27 1.27)
+				)
+			)
+		)
+		(pin "1"
+		)
+		(pin "5"
+		)
+		(pin "4"
+		)
+		(pin "3"
+		)
+		(pin "2"
+		)
+		(pin "6"
+		)
+		(instances
+			(project "Esp32 Can+IMU"
+				(path "/904515b0-f96e-4935-be8a-ac627093fee4"
+					(reference "U7")
+					(unit 1)
+				)
+			)
+		)
+	)
+	(symbol
 		(lib_id "Device:R_US")
 		(at 419.1 459.74 180)
@@
 					(unit 1)
 				)
-			)
-		)
-	)
-	(symbol
-		(lib_id "Power_Protection:USBLC6-2SC6")
-		(at 260.35 292.1 0)
-		(unit 1)
-		(body_style 1)
-		(exclude_from_sim no)
-		(in_bom yes)
-		(on_board yes)
-		(in_pos_files yes)
-		(dnp no)
-		(fields_autoplaced yes)
-		(property "Reference" "U6"
-			(at 262.0011 284.48 0)
-			(show_name no)
-			(do_not_autoplace no)
-			(effects
-				(font
-					(size 1.27 1.27)
-				)
-				(justify left)
-			)
-		)
-		(property "Value" "USBLC6-2SC6"
-			(at 262.0011 287.02 0)
-			(show_name no)
-			(do_not_autoplace no)
-			(effects
-				(font
-					(size 1.27 1.27)
-				)
-				(justify left)
-			)
-		)
-		(property "Footprint" "Package_TO_SOT_SMD:SOT-666"
-			(at 261.62 298.45 0)
-			(hide yes)
-			(show_name no)
-			(do_not_autoplace no)
-			(effects
-				(font
-					(size 1.27 1.27)
-					(italic yes)
-				)
-				(justify left)
-			)
-		)
-		(property "Datasheet" "https://www.st.com/resource/en/datasheet/usblc6-2.pdf"
-			(at 261.62 300.355 0)
-			(hide yes)
-			(show_name no)
-			(do_not_autoplace no)
-			(effects
-				(font
-					(size 1.27 1.27)
-				)
-				(justify left)
-			)
-		)
-		(property "Description" "Very low capacitance ESD protection diode, 2 data-line, SOT-23-6"
-			(at 260.35 292.1 0)
-			(hide yes)
-			(show_name no)
-			(do_not_autoplace no)
-			(effects
-				(font
-					(size 1.27 1.27)
-				)
-			)
-		)
-		(pin "1"
-		)
-		(pin "2"
-		)
-		(pin "3"
-		)
-		(pin "4"
-		)
-		(pin "5"
-		)
-		(pin "6"
-		)
-		(instances
-			(project "Esp32 Can+IMU"
-				(path "/904515b0-f96e-4935-be8a-ac627093fee4"
-					(reference "U6")
-					(unit 1)
-				)
